File: Fan.sch (KiCad schematic (older format))
At the start: 11 parts, among them Q2 DMN65D8L-7, Q3 AOD476, Q4 AOD476, U3 MCP4801, U4 OPA4170

Commit message: Layout sessions 1-4.
Connections:
- net AGND: now also U3.7 (Vss)
- net at R9.2, U4.5 (+): now also Q2.2 (D)
- net +12V renamed FE_V+
- net -12V renamed FE_V-
Other:
- note removed: "Should this be a different ground?"
Changed lines of the file:
@@
-	1    0    0    -1
-$EndComp
-$Comp
-L AGND #PWR059
-U 1 1 52F62EF1
-P 7850 6100
-F 0 "#PWR059" H 7850 6100 40  0001 C CNN
-F 1 "AGND" H 7850 6030 50  0000 C CNN
-F 2 "" H 7850 6100 60  0000 C CNN
-F 3 "" H 7850 6100 60  0000 C CNN
-	1    7850 6100
 	1    0    0    -1
 $EndComp
@@
 Wire Wire Line
 	5900 3750 6050 3750
-$Comp
-L +12V #PWR060
-U 1 1 52F62F17
-P 6450 3050
-F 0 "#PWR060" H 6450 3000 20  0001 C CNN
-F 1 "+12V" H 6450 3150 30  0000 C CNN
-F 2 "" H 6450 3050 60  0000 C CNN
-F 3 "" H 6450 3050 60  0000 C CNN
-	1    6450 3050
-	1    0    0    -1
-$EndComp
 Wire Wire Line
 	6450 3250 6450 3050
-$Comp
-L -12V #PWR061
-U 1 1 52F62F30
-P 6450 4150
-F 0 "#PWR061" H 6450 4280 20  0001 C CNN
-F 1 "-12V" H 6450 4250 30  0000 C CNN
-F 2 "" H 6450 4150 60  0000 C CNN
-F 3 "" H 6450 4150 60  0000 C CNN
-	1    6450 4150
-	-1   0    0    1
-$EndComp
 Wire Wire Line
 	6450 4050 6450 4150
-$Comp
-L AGND #PWR062
-U 1 1 52F62FD1
-P 5450 4550
-F 0 "#PWR062" H 5450 4550 40  0001 C CNN
-F 1 "AGND" H 5450 4480 50  0000 C CNN
-F 2 "" H 5450 4550 60  0000 C CNN
-F 3 "" H 5450 4550 60  0000 C CNN
-	1    5450 4550
-	1    0    0    -1
-$EndComp
-Wire Wire Line
-	5450 4300 5450 4550
 Text HLabel 2700 4800 0    60   Output ~ 0
 CURR_MEAS
@@
 Wire Wire Line
 	4300 4100 4300 4650
-Wire Wire Line
-	5450 3950 5450 3550
 Connection ~ 5450 3550
 Wire Wire Line
@@
 FAN_MODE
 $Comp
-L +12C #PWR063
+L +12C #PWR050
 U 1 1 52F96856
 P 7850 1200
-F 0 "#PWR063" H 7850 1170 30  0001 C CNN
+F 0 "#PWR050" H 7850 1170 30  0001 C CNN
 F 1 "+12C" H 7850 1310 40  0000 C CNN
 F 2 "" H 7850 1200 60  0000 C CNN
@@
 $EndComp
 $Comp
-L AGND #PWR064
-U 1 1 530AD6DD
-P 2750 2750
-F 0 "#PWR064" H 2750 2750 40  0001 C CNN
-F 1 "AGND" H 2750 2680 50  0000 C CNN
-F 2 "" H 2750 2750 60  0000 C CNN
-F 3 "" H 2750 2750 60  0000 C CNN
-	1    2750 2750
-	1    0    0    -1
-$EndComp
-$Comp
-L +5V #PWR065
+L +5V #PWR051
 U 1 1 530AD6E3
 P 3450 2350
-F 0 "#PWR065" H 3450 2440 20  0001 C CNN
+F 0 "#PWR051" H 3450 2440 20  0001 C CNN
 F 1 "+5V" H 3450 2440 30  0000 C CNN
 F 2 "" H 3450 2350 60  0000 C CNN
@@
 	3300 2550 3450 2550
 Connection ~ 3450 2550
-Wire Wire Line
-	2900 2550 2750 2550
-Wire Wire Line
-	2750 2550 2750 2750
 $Comp
 L C C13
@@
 	0    -1   -1   0
 $EndComp
-$Comp
-L AGND #PWR066
-U 1 1 530A4A36
-P 8700 1600
-F 0 "#PWR066" H 8700 1600 40  0001 C CNN
-F 1 "AGND" H 8700 1530 50  0000 C CNN
-F 2 "" H 8700 1600 60  0000 C CNN
-F 3 "" H 8700 1600 60  0000 C CNN
-	1    8700 1600
-	1    0    0    -1
-$EndComp
 Wire Wire Line
 	8100 1300 7850 1300
 Connection ~ 7850 1300
-Wire Wire Line
-	8500 1300 8700 1300
-Wire Wire Line
-	8700 1300 8700 1600
-Text Notes 8850 1500 0    60   ~ 0
-Should this be a different ground?
-Text Notes 8350 6000 0    60   ~ 0
-Should this be a different ground?
 $Comp
 L MOS_N_NUM Q3
@@
 	1    0    0    -1
 $EndComp
+$Comp
+L FE_V+ #PWR052
+U 1 1 53123748
+P 6450 3050
+F 0 "#PWR052" H 6450 3150 30  0001 C CNN
+F 1 "FE_V+" H 6450 3150 30  0000 C CNN
+F 2 "" H 6450 3050 60  0000 C CNN
+F 3 "" H 6450 3050 60  0000 C CNN
+	1    6450 3050
+	1    0    0    -1
+$EndComp
+$Comp
+L FE_V- #PWR64
+U 1 1 5312374E
+P 6450 4150
+F 0 "#PWR64" H 6450 4350 40  0001 C CNN
+F 1 "FE_V-" H 6450 4300 40  0000 C CNN
+F 2 "" H 6450 4150 60  0000 C CNN
+F 3 "" H 6450 4150 60  0000 C CNN
+	1    6450 4150
+	-1   0    0    1
+$EndComp
+Wire Wire Line
+	5450 4550 5450 4300
+Wire Wire Line
+	8700 1600 8700 1300
+Wire Wire Line
+	8700 1300 8500 1300
+Wire Wire Line
+	2750 2750 2750 2550
+Wire Wire Line
+	2750 2550 2900 2550
+Wire Wire Line
+	3450 4400 3450 4300
+Wire Wire Line
+	5450 3900 5450 3550
+$Comp
+L AGND #PWR053
+U 1 1 5313E2E9
+P 3450 4400
+F 0 "#PWR053" H 3450 4400 40  0001 C CNN
+F 1 "AGND" H 3450 4330 50  0000 C CNN
+F 2 "" H 3450 4400 60  0000 C CNN
+F 3 "" H 3450 4400 60  0000 C CNN
+	1    3450 4400
+	1    0    0    -1
+$EndComp
+$Comp
+L AGND #PWR054
+U 1 1 5313E2FB
+P 2750 2750
+F 0 "#PWR054" H 2750 2750 40  0001 C CNN
+F 1 "AGND" H 2750 2680 50  0000 C CNN
+F 2 "" H 2750 2750 60  0000 C CNN
+F 3 "" H 2750 2750 60  0000 C CNN
+	1    2750 2750
+	1    0    0    -1
+$EndComp
+$Comp
+L AGND #PWR055
+U 1 1 5313E306
+P 5450 4550
+F 0 "#PWR055" H 5450 4550 40  0001 C CNN
+F 1 "AGND" H 5450 4480 50  0000 C CNN
+F 2 "" H 5450 4550 60  0000 C CNN
+F 3 "" H 5450 4550 60  0000 C CNN
+	1    5450 4550
+	1    0    0    -1
+$EndComp
+$Comp
+L AGND #PWR056
+U 1 1 5313E311
+P 7850 6100
+F 0 "#PWR056" H 7850 6100 40  0001 C CNN
+F 1 "AGND" H 7850 6030 50  0000 C CNN
+F 2 "" H 7850 6100 60  0000 C CNN
+F 3 "" H 7850 6100 60  0000 C CNN
+	1    7850 6100
+	1    0    0    -1
+$EndComp
+$Comp
+L AGND #PWR057
+U 1 1 5313E31E
+P 8700 1600
+F 0 "#PWR057" H 8700 1600 40  0001 C CNN
+F 1 "AGND" H 8700 1530 50  0000 C CNN
+F 2 "" H 8700 1600 60  0000 C CNN
+F 3 "" H 8700 1600 60  0000 C CNN
+	1    8700 1600
+	1    0    0    -1
+$EndComp
